File: pcb/lcd_test_board/lcd_test_board.kicad_pcb (KiCad board)
At the start: 2 copper layers, 43.2 x 47 mm, 57 parts, among them IC1 LD1117S18TR, IC2 LD1117S33TR, IC3 TPS61041-, J1 FH35W-31S, J2 SAMTEC_BTH-060-01-L-D-A, J3 TS_FPC

Commit message: pcb/lcd_test_board: update
Parts:
- moved R2 6.50 mm to (97.8, 83.8)
- moved R3 6.50 mm to (97.8, 82.2)
- moved R4 6.50 mm to (97.8, 83.8)
- moved R5 6.50 mm to (94.2, 83.7)
- moved R6 6.50 mm to (94.2, 82.2)
- moved R7 6.50 mm to (97.8, 82.2)
- moved R14 6.50 mm to (97.5, 90.2)
- moved R15 6.50 mm to (97.5, 88.8)
- moved R16 6.50 mm to (97.5, 90.2)
- moved R17 6.50 mm to (94.0, 90.2)
- moved R18 6.50 mm to (94.0, 88.7)
- moved R19 6.50 mm to (97.5, 88.7)
Connections:
- J2 pad 31: /DSI_LP_P0 -> /DSI_CLK_LP_P
- J2 pad 33: /DSI_LP_N0 -> /DSI_CLK_LP_N
- J2 pad 35: /DSI_HS_P0 -> /DSI_CLK_P_1
- J2 pad 37: /DSI_HS_N0 -> /DSI_CLK_N_1
- J2 pad 51: /DSI_CLK_LP_P -> /DSI_LP_P0
- J2 pad 53: /DSI_CLK_LP_N -> /DSI_LP_N0
- J2 pad 55: /DSI_CLK_P_1 -> /DSI_HS_P0
- J2 pad 57: /DSI_CLK_N_1 -> /DSI_HS_N0
- R14 pad 2: /DSI_L2_P -> /DSI_CLK_P
- R15 pad 2: /DSI_L2_N -> /DSI_CLK_N
- R16 pad 2: /DSI_L2_P -> /DSI_CLK_P
- R17 pad 1: /DSI_L2_P -> /DSI_CLK_P
- R18 pad 2: /DSI_L2_N -> /DSI_CLK_N
- R19 pad 1: /DSI_L2_N -> /DSI_CLK_N
- R2 pad 2: /DSI_CLK_P -> /DSI_L2_P
- R3 pad 2: /DSI_CLK_N -> /DSI_L2_N
- R4 pad 2: /DSI_CLK_P -> /DSI_L2_P
- R5 pad 1: /DSI_CLK_P -> /DSI_L2_P
- R6 pad 2: /DSI_CLK_N -> /DSI_L2_N
- R7 pad 1: /DSI_CLK_N -> /DSI_L2_N
Routing:
- net /DSI_LP_P0: track 6.33 -> 8.13 mm
- net /DSI_CLK_LP_P: track 8.13 -> 6.33 mm
- net /DSI_HS_N0: track 2.66 -> 4.07 mm
- net /DSI_CLK_N_1: track 4.07 -> 2.66 mm
