File: pcb/lcd_test_board/myir_connector.sch (KiCad schematic (older format))
At the start: 1 part, among them J2 SAMTEC_BTH-060-01-L-D-A

Commit message: pcb/lcd_test_board: update
Changed lines of the file:
@@
 $Descr A4 11693 8268
 encoding utf-8
-Sheet 7 8
+Sheet 8 8
 Title ""
 Date ""
@@
 Wire Wire Line
 	5800 2800 7650 2800
-Text HLabel 7650 2700 2    50   Output ~ 0
-DSI_LP_N0
-Text HLabel 7650 2600 2    50   Output ~ 0
-DSI_LP_P0
-Text HLabel 7650 2900 2    50   Output ~ 0
-DSI_HS_N0
 Wire Wire Line
 	5800 2700 7650 2700
@@
 Wire Wire Line
 	5800 2600 7650 2600
-Text HLabel 7650 2800 2    50   Output ~ 0
-DSI_HS_P0
 Text HLabel 7650 3300 2    50   Output ~ 0
 DSI_HS_P1
@@
 Wire Wire Line
 	5800 3300 7650 3300
-Text HLabel 7650 3600 2    50   Output ~ 0
-DSI_CLK_LP_P
-Text HLabel 7650 3700 2    50   Output ~ 0
-DSI_CLK_LP_N
-Text HLabel 7650 3800 2    50   Output ~ 0
-DSI_CLK_P
-Text HLabel 7650 3900 2    50   Output ~ 0
-DSI_CLK_N
 Wire Wire Line
 	5800 3600 7650 3600
@@
 Wire Wire Line
 	3250 1700 5100 1700
+Text HLabel 7650 2900 2    50   Output ~ 0
+DSI_CLK_N
+Text HLabel 7650 2800 2    50   Output ~ 0
+DSI_CLK_P
+Text HLabel 7650 2700 2    50   Output ~ 0
+DSI_CLK_LP_N
+Text HLabel 7650 2600 2    50   Output ~ 0
+DSI_CLK_LP_P
+Text HLabel 7650 3800 2    50   Output ~ 0
+DSI_HS_P0
+Text HLabel 7650 3900 2    50   Output ~ 0
+DSI_HS_N0
+Text HLabel 7650 3600 2    50   Output ~ 0
+DSI_LP_P0
+Text HLabel 7650 3700 2    50   Output ~ 0
+DSI_LP_N0
 $EndSCHEMATC
